File: PDU_E4.kicad_sch (KiCad schematic)
At the start: 5 parts

Commit message: VER1.0: внес исправления замечаний
Parts:
- added F1, F2: Fuse, symbol Device:Fuse
Connections:
- net Channel_1: now also F2.2; no longer D2.A2, D3.A2
- net Channel_2: now also F1.2; no longer D4.A2, D5.A2
- new net: D2.A2, D3.A2, F2.1
- new net: D4.A2, D5.A2, F1.1
Other:
- note added: "X2"
- note added: "X3"
- note added: "X4"
- note added: "X5"
- note added: "X6"
- note added: "X7"

Commit message: VER1: сделал таблицу и шины
Parts:
- renumbered D5 to K1, D4 to K2, D3 to K3, D2 to K4, D1 to K5
Other:
- note added: "U1"
- note added: "А3.1"
- note added: "А3.2"
- note added: "А3.3"
- note added: "НВЦТ.0001.0400.100"
- note added: "ООО "Электротранспортные"
- note added: "технологии""
- note removed: "А1"
- note removed: "А2"
- note removed: "А4"
- company: ООО "Электротранспортные технологии" -> (none)

Commit message: VER1: готово
Other:
- note added: "1. Использовать шины сечением 3х15мм."
- note added: "2. Для внутренних электрических соединений использовать провод ММП (АМП)-H50-0.35."
Changed lines of the file:
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@@
 		)
 	)
+	(text "1. Использовать шины сечением 3х15мм.\n"
+		(exclude_from_sim no)
+		(at 393.7 174.498 0)
+		(effects
+			(font
+				(size 2.5 2.5)
+			)
+			(justify left)
+		)
+	)
 	(text "X7"
 		(exclude_from_sim no)
@@
 		)
 	)
+	(text "2. Для внутренних электрических соединений использовать провод ММП (АМП)-H50-0.35."
+		(exclude_from_sim no)
+		(at 393.7 179.07 0)
+		(effects
+			(font
+				(size 2.5 2.5)
+			)
+			(justify left)
+		)
+	)
 	(text "X5"
 		(exclude_from_sim no)
@@
 				(font
 					(size 5 5)
+					(color 0 0 0 1)
 				)
 			)
@@
 				(font
 					(size 3.5 3.5)
+					(color 0 0 0 1)
 				)
 				(justify right)
@@
 				(font
 					(size 3.5 3.5)
+					(color 0 0 0 1)
 				)
 				(justify right)
@@
 				(font
 					(size 5 5)
+					(color 0 0 0 1)
 				)
 			)
@@
 				(font
 					(size 3.5 3.5)
+					(color 0 0 0 1)
 				)
 				(justify right)
@@
 				(font
 					(size 3.5 3.5)
+					(color 0 0 0 1)
 				)
 				(justify right)
@@
 				(font
 					(size 3.5 3.5)
+					(color 0 0 0 1)
 				)
 				(justify right)
